File: COMPRESSORFOC.kicad_pcb (KiCad board)
At the start: 2 copper layers, 135 x 135 mm, 90 parts, among them J1 ESP32-PICO-KIT_ESP32-PICO-KIT, J10 3.3V, J11 Pin 1, J12 Pin 2, J13 GND, J2 Fan 1+, J3 Fan 1-, J4 15V+, J5 15VGND, J6 Conn_01x03_Socket, J7 Conn_01x03_Socket, J8 Fan 2+, J9 Fan 2-, Q1 NMOSIPD50R280CEAUMA1, U2 INA240A2DR, U3 INA240A2DR, U5 INA240A2DR

Commit message: revised driver
Parts:
- removed the C10 at (158.6, 103.1)
- removed the C29 at (182.7, 77.8)
- removed the C3 at (159.2, 114.9)
- removed the C31 at (163.6, 55.8)
- removed the C4 at (159.1, 107.7)
- removed the C6 at (159.2, 112.5)
- removed the C7 at (159.0, 105.7)
- removed the C9 at (159.3, 110.1)
- removed the R1 at (152.2, 107.1)
- removed the R10 at (110.5, 120.5)
- removed the R11 at (158.7, 118.7)
- removed the R2 at (156.4, 113.0)
- removed R23: 100, Resistor_SMD:R_0603_1608Metric_Pad0.98x0.95mm_HandSolder
- removed the R3 at (155.6, 109.4)
- removed the R5 at (157.9, 116.6)
- removed the R7 at (153.4, 102.6)
- added C30: 1u, Capacitor_SMD:C_2225_5664Metric_Pad1.80x6.60mm_HandSolder, F.Cu at (200.7, 74.9)
- added C8: 2n, Capacitor_SMD:C_0603_1608Metric_Pad1.08x0.95mm_HandSolder, F.Cu at (143.7, 141.2)
- added D1: CLV1L-FKB, LED_SMD:LED_Cree-PLCC4_3.2x2.8mm_CCW, F.Cu at (103.9, 119.8)
- added D2: CLV1L-FKB, LED_SMD:LED_Cree-PLCC4_3.2x2.8mm_CCW, F.Cu at (103.9, 126.7)
- added D3: S10JC-HF, Diode_SMD:D_SMC_Handsoldering, F.Cu at (127.5, 62.4)
- added R17: 47k, Resistor_SMD:R_2512_6332Metric_Pad1.40x3.35mm_HandSolder, F.Cu at (173.6, 29.4)
- added R18: 47k, Resistor_SMD:R_2512_6332Metric_Pad1.40x3.35mm_HandSolder, F.Cu at (200.2, 55.3)
- added R19: 47k, Resistor_SMD:R_2512_6332Metric_Pad1.40x3.35mm_HandSolder, F.Cu at (202.8, 29.6)
- added TH1: Thermistor_NTC, COMPRESSORFOC:NTC_compressorfoc, F.Cu at (116.2, 100.7)
- ?: value (none) -> standoff hole; footprint (none) -> COMPRESSORFOC:standoff hole
- C31: renamed from C30; footprint Capacitor_SMD:C_1812_4532Metric_Pad1.57x3.40mm_HandSolder -> Capacitor_SMD:C_2225_5664Metric_Pad1.80x6.60mm_HandSolder
- D5: renamed from D2; footprint COMPRESSORFOC:TO-252-2_DiodeFOCCustom -> COMPRESSORFOC:TO-263-2-FOC
- J12: renamed from J6; footprint COMPRESSORFOC:TerminalBlock3pin -> COMPRESSORFOC:IEC_plugin
- J9: renamed from J5; value 15VGND -> 15V-
- R4: value 100 -> 1M; footprint Resistor_SMD:R_0603_1608Metric_Pad0.98x0.95mm_HandSolder -> Resistor_SMD:R_0805_2012Metric_Pad1.20x1.40mm_HandSolder
- moved J12 47.9 mm to (83.0, 104.8)
- moved R4 39.2 mm to (142.6, 143.6), turned to 180 degrees
- moved R5 22.2 mm to (149.9, 140.1), turned to -90 degrees
- moved C2 21.9 mm to (137.4, 132.9), turned to 180 degrees
- moved C19 14.5 mm to (175.5, 123.5), turned to 0 degrees
- moved C25 7.45 mm to (168.5, 31.7)
- moved C27 6.64 mm to (197.6, 31.1)
- moved C15 6.56 mm to (159.8, 109.2)
- moved C20 5.98 mm to (164.2, 122.0), turned to -90 degrees
- moved C10 4.43 mm to (169.7, 122.2), turned to -90 degrees
- moved D4 4.38 mm to (151.8, 31.2)
- moved D5 3.66 mm to (158.7, 41.2)
- moved C14 2.80 mm to (168.1, 122.2), turned to -90 degrees
- moved R6 2.67 mm to (150.2, 101.5), turned to 180 degrees
- moved C9 2.65 mm to (166.2, 122.2), turned to -90 degrees
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- renumbered C32 to C1, C11 to C10, C12 to C11, C13 to C12, C14 to C13, C15 to C14, C16 to C15, C17 to C16, C18 to C17, C19 to C18, C20 to C19, C35 to C2, C21 to C20, C36 to C21, C37 to C22, C22 to C23, C23 to C24, C24 to C25, C25 to C26, C26 to C27, C27 to C28, C28 to C29, C33 to C3, C38 to C32, C34 to C4, C1 to C5, C2 to C6, C5 to C7, C8 to C9, D1 to D4, J8 to J10, J9 to J11, J7 to J13, J11 to J2, J13 to J3, J2 to J4, J3 to J5, J10 to J6, J12 to J7, J4 to J8, R6 to R1, R17 to R10, R15 to R11, R19 to R12, R20 to R13, R21 to R14, R22 to R15, R24 to R16, R9 to R2, R8 to R3, R12 to R5, R13 to R6, R14 to R7, R16 to R8, R18 to R9
Connections:
- BridgeRectifier1 pad 3: Line 2 -> Net-(BridgeRectifier1-Line_2)
- BridgeRectifier1 pad 4: V- -> Net-(BridgeRectifier1-V-)
- C20 pad 1: Net-(U1-VFO) -> VOT
- J1 pad J2_16: ExtraPin2 -> Net-(J1-IO38)
- J1 pad J2_17: unconnected-(J1-IO37-PadJ2_17) -> VFO
- J1 pad J3_10: Net-(J1-IO27) -> LIN(U)
- J1 pad J3_11: Net-(J1-IO14) -> HIN(U)
- J1 pad J3_14: Net-(J1-IO15) -> ExtraPin2
- J1 pad J3_15: Net-(J1-IO2) -> unconnected-(J1-IO2-PadJ3_15)
- J1 pad J3_16: Net-(J1-IO4) -> unconnected-(J1-IO4-PadJ3_16)
- J1 pad J3_4: unconnected-(J1-SENSOR_VP-PadJ3_4) -> Net-(J1-SENSOR_VP)
- J1 pad J3_5: unconnected-(J1-SENSOR_VN-PadJ3_5) -> Net-(J1-SENSOR_VN)
- J1 pad J3_6: Net-(J1-IO25) -> LIN(W)
- J1 pad J3_7: Net-(J1-IO26) -> HIN(W)
- J1 pad J3_8: Net-(J1-IO32) -> LIN(V)
- J1 pad J3_9: Net-(J1-IO33) -> HIN(V)
- J12 pad 3: V- -> Earth Ground
- J5 pad 1: /Fan 1- -> GND
- R1 pad 1: Net-(J1-IO15) -> Net-(J1-SENSOR_VN)
- R2 pad 1: Net-(J1-IO2) -> Net-(J1-SENSOR_VP)
- R3 pad 1: Net-(J1-IO4) -> Net-(J1-IO38)
- R4 pad 1: Net-(J1-IO26) -> VFO
- R4 pad 2: HIN(W) -> V3.3
- R6 pad 2: V- -> Net-(BridgeRectifier1-V-)
- R7 pad 2: V- -> Net-(BridgeRectifier1-V-)
- U1 pad 16: Net-(U1-VFO) -> VFO
- U4 pad 8: VLine -> Net-(D3-K)
Routing:
- net Net-(J1-IO4): track 47.0 -> 0.00 mm, vias 2 -> 0
- net VFO: track 0.00 -> 46.3 mm, vias 0 -> 2
- net Net-(J1-IO38): track 0.00 -> 44.3 mm
- net 15VLine: track 153.6 -> 196.9 mm, vias 2 -> 0
- net Net-(J1-IO2): track 41.5 -> 0.00 mm, vias 1 -> 0
- net Net-(J1-IO26): track 39.9 -> 0.00 mm, vias 1 -> 0
- net Net-(J1-IO15): track 39.4 -> 0.00 mm, vias 2 -> 0
- net V-: track 37.2 -> 0.00 mm, vias 1 -> 0
- net Net-(BridgeRectifier1-V-): track 0.00 -> 37.2 mm, vias 0 -> 1
- net Net-(J1-IO14): track 30.9 -> 0.00 mm
- net Net-(J1-IO25): track 28.9 -> 0.00 mm
- net HIN(W): track 11.9 -> 40.1 mm
- net Net-(J1-IO33): track 27.2 -> 0.00 mm, vias 1 -> 0
- net Net-(J1-IO32): track 27.0 -> 0.00 mm
- net Net-(J1-IO27): track 25.6 -> 0.00 mm
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- added copper zone on B.Cu, net Line 1
- added copper zone on B.Cu, net Line 2
- added copper zone on B.Cu, net Net-(BridgeRectifier1-Line_2)
- added copper zone on F.Cu, net Net-(BridgeRectifier1-V-)
- removed copper zone on F.Cu, net Line 1
- removed copper zone on F.Cu, net Line 2
- removed copper zone on F.Cu, net V-
Other:
- outline, holes or cut-outs redrawn
- board text added: "15V+"
- board text added: "15V-"
- board text added: "Earth GND"
- board text added: "Fan 1+"
- board text added: "Fan 1-"
- board text added: "Fan 2+"
- board text added: "Fan 2-"
- board text added: "Line"
- board text added: "Neutral"
- board text removed: "AC IN"
- board text removed: "GND"
